Commit message: added training data generation algorithm

File: models/zephyr_delta_wing_ardupilot_camera/delta_wing_t.urdf (robot description, URDF)
Before this commit: robot zephyr_delta_wing_ardupilot_camera, 16 links, 15 joints
Links:
- removed link zephyr_delta_wing_ardupilot_camera__zephyr_delta_wing_rudder__base_link
Joints:
- removed joint zephyr_delta_wing_ardupilot_camera__zephyr_delta_wing_rudder__base_link_joint
- joint zephyr_delta_wing_ardupilot_camera__camera_mount: origin xyz=0      -0.34     0.05423 rpy=0       0      -1.57079 -> xyz=0   -0.34  0.28 rpy=0       0      -1.57079
- joint zephyr_delta_wing_ardupilot_camera__camera_pole_joint: origin xyz=0      -0.4     -0.02577 rpy=-1.57079  1.57079  3.14159 -> xyz=0  -0.4  0.2 rpy=-1.57079  1.57079  3.14159
- joint zephyr_delta_wing_ardupilot_camera__skid_pad_joint: origin xyz=0      -0.07    -0.24577 rpy=0 0 0 -> xyz=0   -0.07 -0.02 rpy=0 0 0
- joint zephyr_delta_wing_ardupilot_camera__virtual_camera_mount: origin xyz=0       0      -0.22577 rpy=0 0 0 -> xyz=0 0 0 rpy=0 0 0
- joint zephyr_delta_wing_ardupilot_camera__zephyr_delta_wing_rudder__flap_left_joint: origin xyz=0.453 0.199 0.007 rpy=0 0 0 -> xyz=0.453   0.199   0.23277 rpy=0 0 0
- joint zephyr_delta_wing_ardupilot_camera__zephyr_delta_wing_rudder__flap_right_joint: origin xyz=-0.453  0.199  0.007 rpy=0 0 0 -> xyz=-0.453    0.199    0.23277 rpy=0 0 0
- joint zephyr_delta_wing_ardupilot_camera__zephyr_delta_wing_rudder__propeller_1_joint: origin xyz=0.35  -0.32   0.008 rpy=0      1.57079 0 -> xyz=0.35    -0.32     0.23377 rpy=0      1.57079 0
- joint zephyr_delta_wing_ardupilot_camera__zephyr_delta_wing_rudder__propeller_2_joint: origin xyz=-0.35  -0.32   0.008 rpy=0      1.57079 0 -> xyz=-0.35    -0.32     0.23377 rpy=0      1.57079 0
- joint zephyr_delta_wing_ardupilot_camera__zephyr_delta_wing_rudder__zephyr/imu_joint: origin xyz=0 0 0 rpy=0 0 0 -> xyz=0      0      0.22577 rpy=0 0 0

File: models/zephyr_delta_wing_rudder/model.urdf (robot description, URDF)
Before this commit: robot zephyr_delta_wing_rudder, 6 links, 5 joints
Links:
- added link zephyr_delta_wing_rudder__base_link, mass 1e-10
Joints:
- added joint zephyr_delta_wing_rudder__base_link_joint: type fixed, parent zephyr_delta_wing_rudder__base_link, child zephyr_delta_wing_rudder__wing, origin xyz=0      0      0.02577 rpy=0 0 0, axis 0 0 0, limit lower=0 upper=0 effort=0 velocity=0
- joint zephyr_delta_wing_rudder__flap_left_joint: origin xyz=0.453   0.199   0.03277 rpy=0 0 0 -> xyz=0.453 0.199 0.007 rpy=0 0 0
- joint zephyr_delta_wing_rudder__flap_right_joint: origin xyz=-0.453    0.199    0.03277 rpy=0 0 0 -> xyz=-0.453  0.199  0.007 rpy=0 0 0
- joint zephyr_delta_wing_rudder__propeller_1_joint: origin xyz=0.35    -0.32     0.03377 rpy=0      1.57079 0 -> xyz=0.35  -0.32   0.008 rpy=0      1.57079 0
- joint zephyr_delta_wing_rudder__propeller_2_joint: origin xyz=-0.35    -0.32     0.03377 rpy=0      1.57079 0 -> xyz=-0.35  -0.32   0.008 rpy=0      1.57079 0
- joint zephyr_delta_wing_rudder__zephyr/imu_joint: origin xyz=0      0      0.02577 rpy=0 0 0 -> xyz=0 0 0 rpy=0 0 0
